Commit message: added moving stereo camera

File: mobile_robot_description/xacro/robot.xacro (robot description, xacro)
@@ -63,69 +63,121 @@
     <xacro:default_inertial mass="20"/>
   </link>
-  <xacro:wheel name="wh_left_back" x="1" y="-1"/>
-  <xacro:wheel name="wh_right_back" x="-1" y="-1"/>
-  <xacro:wheel name="wh_left_front" x="1" y="1"/>
-  <xacro:wheel name="wh_right_front" x="-1" y="1"/>
-  <!-- =================== Kinect ==================== -->
-  <link name="kinect_link">
-    <visual>
-      <origin xyz="0 0 0" rpy="0 0 0"/>
-      <geometry>
-        <mesh filename="package://mobile_robot_description/meshes/kinect.stl" scale="0.01 0.01 0.01"/>
-      </geometry>
-      <material name="kinect">
-        <color rgba="1 0.9 0.9 1"/>
-      </material>
+  <joint name="cam_stand_joint" type="fixed">
+    <origin xyz="0.0 0.0 0.45" rpy="0 0 0" />
+    <parent link="base_link"/>
+    <child link="cam_stand" />
+  </joint>
+  <!-- the model -->
+  <link name="cam_stand">
+    <inertial>
+      <mass value="1" />
+      <origin xyz="0 0 0.00" />
+      <inertia ixx="1.0" ixy="0.0" ixz="0.0"
+        iyy="1.0" iyz="0.0"
+        izz="1.0" />
+    </inertial>
+    <visual>
+      <geometry>
+        <box size=".1 .1 .9" /> <!-- does not need to match collision -->
+      </geometry>
     </visual>
     <collision>
       <origin xyz="0 0 0" rpy="0 0 0"/>
       <geometry>
-        <box size="0.28 0.07 0.08"/>
+        <box size="0.6 0.4 0.10"/>
       </geometry>
     </collision>
-    <xacro:default_inertial mass="0.2"/>
-  </link>
-  <joint name="base_link_kinect_link" type="fixed">
-    <origin xyz="0.265 0 0.087" rpy="0 0 ${pi/2}"/>
-    <parent link="base_link"/>
-    <child link="kinect_link"/>
-  </joint>
-  <!-- =================== Gazebo - Kinect ==================== -->
-  <link name="gz_kinect_link">
-    <visual>
-      <origin xyz="0 0 0" rpy="0 0 0"/>
-      <geometry>
-        <sphere radius="0.05"/>
-      </geometry>
-      <material name="kinect">
-        <color rgba="1 0.9 0.9 1"/>
-      </material>
-    </visual>
-    <collision>
-      <origin xyz="0 0 0" rpy="0 0 0"/>
-      <geometry>
-        <sphere radius="0.05"/>
-      </geometry>
-    </collision>
-    <xacro:default_inertial mass="0.2"/>
-  </link>
-  <joint name="kinect_link_gz_kinect_link" type="fixed">
-    <origin xyz="0 0 0" rpy="0 0 -${pi/2}"/>
-    <parent link="kinect_link"/>
-    <child link="gz_kinect_link"/>
-  </joint>
-  <gazebo reference="gz_kinect_link">
-    <sensor type="depth" name="kinect">
+  </link>
+   <joint name="cam_prismatic" type="prismatic">
+      <child link="cam_stand_primsatic" />
+      <parent link="cam_stand"/>
+      <origin xyz="0.0 0 0.475" rpy="0 0 0"/>
+      <axis xyz="0 0 -1"/>
+      <limit effort="1000.0" lower="-0.2" upper="0.2" velocity="0.5"/>
+    </joint>
+  <transmission name="cam_prismatic_trans">
+    <type>transmission_interface/SimpleTransmission</type>
+    <joint name="cam_prismatic">
+      <hardwareInterface>hardware_interface/EffortJointInterface</hardwareInterface>
+    </joint>
+    <actuator name="motorToCamPris">
+      <hardwareInterface>hardware_interface/EffortJointInterface</hardwareInterface>
+      <mechanicalReduction>1</mechanicalReduction>
+    </actuator>
+  </transmission>
+  <link name="cam_stand_primsatic">
+    <inertial>
+      <mass value=".1" />
+      <origin xyz="0 0 0.00" />
+      <inertia ixx="1.0" ixy="0.0" ixz="0.0"
+        iyy="1.0" iyz="0.0"
+        izz="1.0" />
+    </inertial>
+    <visual>
+      <geometry>
+        <box size="0.01 0.01 0.01" /> <!-- does not need to match collision -->
+      </geometry>
+    </visual>
+  </link>
+   <joint name="cam_revolute" type="continuous">
+      <origin xyz="0.0 0.0 0.0" rpy="0 0 0"/>
+      <axis rpy="0 0 0" xyz="0 1 0"/>
+      <parent link="cam_stand_primsatic"/>
+      <child link="cam"/>
+    </joint>
+  <transmission name="cam_revolute_trans">
+    <type>transmission_interface/SimpleTransmission</type>
+    <joint name="cam_revolute">
+      <hardwareInterface>hardware_interface/EffortJointInterface</hardwareInterface>
+    </joint>
+    <actuator name="motorToCamRev">
+      <hardwareInterface>hardware_interface/EffortJointInterface</hardwareInterface>
+      <mechanicalReduction>1</mechanicalReduction>
+    </actuator>
+  </transmission>
+  <link name="cam">
+    <inertial>
+      <mass value=".1" />
+      <origin xyz="0 0 0.00" />
+      <inertia ixx="1.0" ixy="0.0" ixz="0.0"
+        iyy="1.0" iyz="0.0"
+        izz="1.0" />
+    </inertial>
+    <visual>
+      <geometry>
+        <box size="0.15 0.15 0.15" /> <!-- does not need to match collision -->
+      </geometry>
+    </visual>
+  </link>
+  <gazebo reference="cam">
+    <gravity>true</gravity>
+    <sensor name="imu_sensor" type="imu">
+      <always_on>true</always_on>
+      <update_rate>100</update_rate>
+      <visualize>true</visualize>
+      <topic>camera_imu</topic>
+      <plugin filename="libgazebo_ros_imu_sensor.so" name="imu_plugin">
+        <topicName>camera_imu</topicName>
+        <bodyName>cam</bodyName>
+        <updateRateHZ>100.0</updateRateHZ>
+        <gaussianNoise>0.001</gaussianNoise>
+        <xyzOffset>0 0 0</xyzOffset>
+        <rpyOffset>0 0 0</rpyOffset>
+        <frameName>cam</frameName>
+        <initialOrientationAsReference>false</initialOrientationAsReference>
+      </plugin>
       <pose>0 0 0 0 0 0</pose>
-      <always_on>1</always_on>
-      <visualize>true</visualize>
-      <camera>
+    </sensor>
+  </gazebo>
+    <gazebo reference="cam">
+    <sensor type="multicamera" name="stereo_camera">
+      <update_rate>30.0</update_rate>
+      <camera name="left">
         <horizontal_fov>1.047</horizontal_fov>
-        <image>
-          <width>640</width>
-          <height>480</height>
-          <format>R8G8B8</format>
-        </image>
-        <depth_camera></depth_camera>
+            <image>
+                <width>640</width>
+                <height>480</height>
+                <format>RGB_INT8</format>
+            </image>
         <clip>
           <near>0.1</near>
@@ -135,32 +187,46 @@
           <type>gaussian</type>
           <mean>0.0</mean>
-          <stddev>0.7</stddev>
+          <stddev>0.0001</stddev>
         </noise>
       </camera>
-      <plugin name="camera_controller" filename="libgazebo_ros_openni_kinect.so">
-        <!-- <baseline>0.2</baseline> -->
+      <camera name="right">
+        <pose>0 -0.1 0 0 0 0</pose>
+        <horizontal_fov>1.047</horizontal_fov>
+            <image>
+                <width>640</width>
+                <height>480</height>
+                <format>RGB_INT8</format>
+            </image>
+        <clip>
+          <near>0.1</near>
+          <far>100</far>
+        </clip>
+        <noise>
+          <type>gaussian</type>
+          <mean>0.0</mean>
+          <stddev>0.0001</stddev>
+        </noise>
+      </camera>
+      <plugin name="stereo_camera_controller" filename="libgazebo_ros_multicamera.so">
         <alwaysOn>true</alwaysOn>
-        <updateRate>10.0</updateRate>
-        <cameraName>kinect_sensor</cameraName>
-        <frameName>gz_kinect_link</frameName>
-        <imageTopicName>/mobile_robot/rgb/image_raw</imageTopicName>
-        <depthImageTopicName>/mobile_robot/depth/image_raw</depthImageTopicName>
-        <pointCloudTopicName>/mobile_robot/depth/points</pointCloudTopicName>
-        <cameraInfoTopicName>/mobile_robot/rgb/camera_info</cameraInfoTopicName>
-        <depthImageInfoTopicName>/mobile_robot/depth/camera_info</depthImageInfoTopicName>
-        <pointCloudCutoff>0.4</pointCloudCutoff>
-        <hackBaseline>0.07</hackBaseline>
-        <distortionK1>0.001</distortionK1>
-        <distortionK2>0.001</distortionK2>
-        <distortionK3>0.001</distortionK3>
-        <distortionT1>0.001</distortionT1>
-        <distortionT2>0.001</distortionT2>
-        <CxPrime>0</CxPrime>
-        <Cx>0</Cx>
-        <Cy>0</Cy>
-        <focalLength>0</focalLength>
+        <updateRate>0.0</updateRate>
+        <cameraName>simulated/camera</cameraName>
+        <imageTopicName>image_raw</imageTopicName>
+        <cameraInfoTopicName>camera_info</cameraInfoTopicName>
+        <frameName>left_camera_optical_frame</frameName>
+        <!--<rightFrameName>right_camera_optical_frame</rightFrameName>-->
+        <hackBaseline>0.1</hackBaseline>
+        <distortionK1>0.0</distortionK1>
+        <distortionK2>0.0</distortionK2>
+        <distortionK3>0.0</distortionK3>
+        <distortionT1>0.0</distortionT1>
+        <distortionT2>0.0</distortionT2>
       </plugin>
     </sensor>
   </gazebo>
+  <xacro:wheel name="wh_left_back" x="1" y="-1"/>
+  <xacro:wheel name="wh_right_back" x="-1" y="-1"/>
+  <xacro:wheel name="wh_left_front" x="1" y="1"/>
+  <xacro:wheel name="wh_right_front" x="-1" y="1"/>
   <!-- =================== Gazebo ==================== -->
   <gazebo>

Commit message: tuned control file

File: mobile_robot_description/xacro/robot.xacro (robot description, xacro)
@@ -30,5 +30,5 @@
     </link>
     <joint name="base_link_${name}" type="continuous">
-      <origin xyz="${y*0.25} ${x*0.25} 0" rpy="0 0 0"/>
+      <origin xyz="${y*0.18} ${x*0.25} 0" rpy="0 0 0"/>
       <axis rpy="0 0 0" xyz="0 1 0"/>
       <parent link="base_link"/>
@@ -49,5 +49,5 @@
       <origin xyz="0 0 0" rpy="0 0 0"/>
       <geometry>
-        <box size="0.6 0.4 0.10"/>
+        <box size="0.35 0.4 0.10"/>
       </geometry>
       <material name="acrylic">
@@ -58,5 +58,5 @@
       <origin xyz="0 0 0" rpy="0 0 0"/>
       <geometry>
-        <box size="0.6 0.4 0.10"/>
+        <box size="0.35 0.4 0.10"/>
       </geometry>
     </collision>

Commit message: added respawn

File: mobile_robot_description/xacro/robot.xacro (robot description, xacro)
@@ -1,48 +1,4 @@
 <?xml version="1.0"?>
 <robot xmlns:xacro="http://www.ros.org/wiki/xacro" name="mobile_robot">
-  <xacro:macro name="default_inertial" params="mass">
-    <inertial>
-      <mass value="${mass}"/>
-      <inertia ixx="1.0" ixy="0.0" ixz="0.0" iyy="1.0" iyz="0.0" izz="1.0"/>
-    </inertial>
-  </xacro:macro>
-  <xacro:macro name="default_inertial" params="mass">
-    <inertial>
-      <mass value="${mass}"/>
-      <inertia ixx="1.0" ixy="0.0" ixz="0.0" iyy="1.0" iyz="0.0" izz="1.0"/>
-    </inertial>
-  </xacro:macro>
-  <xacro:macro name="wheel" params="name x y">
-    <link name="${name}">
-      <visual>
-        <origin xyz="0 0 0" rpy="${pi/2} 0 0"/>
-        <geometry>
-          <cylinder length="0.04" radius="0.1"/>
-        </geometry>
-      </visual>
-      <collision>
-        <origin xyz="0 0 0" rpy="${pi/2} 0 0"/>
-        <geometry>
-          <cylinder length="0.04" radius="0.1"/>
-        </geometry>
-      </collision>
-      <xacro:default_inertial mass="0.6"/>
-    </link>
-    <joint name="base_link_${name}" type="continuous">
-      <origin xyz="${y*0.25} ${x*0.25} 0" rpy="0 0 0"/>
-      <axis rpy="0 0 0" xyz="0 1 0"/>
-      <parent link="base_link"/>
-      <child link="${name}"/>
-    </joint>
-    <transmission name="base_link_${name}_wheel_trans">
-      <type>transmission_interface/SimpleTransmission</type>
-      <actuator name="base_link_${name}_wheel_motor">
-        <mechanicalReduction>1</mechanicalReduction>
-      </actuator>
-      <joint name="base_link_${name}">
-        <hardwareInterface>hardware_interface/VelocityJointInterface</hardwareInterface>
-      </joint>
-    </transmission>
-  </xacro:macro>
   <link name="base_link">
     <visual>
@@ -61,5 +17,8 @@
       </geometry>
     </collision>
-    <xacro:default_inertial mass="20"/>
+    <inertial>
+      <mass value="20.0"/>
+      <inertia ixx="1.0" ixy="0.0" ixz="0.0" iyy="1.0" iyz="0.0" izz="1.0"/>
+    </inertial>
   </link>
   <joint name="cam_stand_joint" type="fixed">
@@ -225,8 +184,136 @@
     </sensor>
   </gazebo>
-  <xacro:wheel name="wh_left_back" x="1" y="-1"/>
-  <xacro:wheel name="wh_right_back" x="-1" y="-1"/>
-  <xacro:wheel name="wh_left_front" x="1" y="1"/>
-  <xacro:wheel name="wh_right_front" x="-1" y="1"/>
+  <link name="wh_left_back">
+    <visual>
+      <origin xyz="0 0 0" rpy="1.57079632679 0 0"/>
+      <geometry>
+        <cylinder length="0.04" radius="0.1"/>
+      </geometry>
+    </visual>
+    <collision>
+      <origin xyz="0 0 0" rpy="1.57079632679 0 0"/>
+      <geometry>
+        <cylinder length="0.04" radius="0.1"/>
+      </geometry>
+    </collision>
+    <inertial>
+      <mass value="1.0"/>
+      <inertia ixx="1.0" ixy="0.0" ixz="0.0" iyy="1.0" iyz="0.0" izz="1.0"/>
+    </inertial>
+  </link>
+  <joint name="base_link_wh_left_back" type="continuous">
+    <origin xyz="-.25 .25 0" rpy="0 0 0"/>
+    <axis rpy="0 0 0" xyz="0 1 0"/>
+    <parent link="base_link"/>
+    <child link="wh_left_back"/>
+  </joint>
+  <transmission name="base_link_wh_left_back_wheel_trans">
+    <type>transmission_interface/SimpleTransmission</type>
+    <actuator name="base_link_wh_left_back_wheel_motor">
+      <mechanicalReduction>1</mechanicalReduction>
+    </actuator>
+    <joint name="base_link_wh_left_back">
+      <hardwareInterface>hardware_interface/VelocityJointInterface</hardwareInterface>
+    </joint>
+  </transmission>
+  <link name="wh_right_back">
+    <visual>
+      <origin xyz="0 0 0" rpy="1.57079632679 0 0"/>
+      <geometry>
+        <cylinder length="0.04" radius="0.1"/>
+      </geometry>
+    </visual>
+    <collision>
+      <origin xyz="0 0 0" rpy="1.57079632679 0 0"/>
+      <geometry>
+        <cylinder length="0.04" radius="0.1"/>
+      </geometry>
+    </collision>
+    <inertial>
+      <mass value="1.0"/>
+      <inertia ixx="1.0" ixy="0.0" ixz="0.0" iyy="1.0" iyz="0.0" izz="1.0"/>
+    </inertial>
+  </link>
+  <joint name="base_link_wh_right_back" type="continuous">
+    <origin xyz="-.25 -.25 0" rpy="0 0 0"/>
+    <axis rpy="0 0 0" xyz="0 1 0"/>
+    <parent link="base_link"/>
+    <child link="wh_right_back"/>
+  </joint>
+  <transmission name="base_link_wh_right_back_wheel_trans">
+    <type>transmission_interface/SimpleTransmission</type>
+    <actuator name="base_link_wh_right_back_wheel_motor">
+      <mechanicalReduction>1</mechanicalReduction>
+    </actuator>
+    <joint name="base_link_wh_right_back">
+      <hardwareInterface>hardware_interface/VelocityJointInterface</hardwareInterface>
+    </joint>
+  </transmission>
+  <link name="wh_left_front">
+    <visual>
+      <origin xyz="0 0 0" rpy="1.57079632679 0 0"/>
+      <geometry>
+        <cylinder length="0.04" radius="0.1"/>
+      </geometry>
+    </visual>
+    <collision>
+      <origin xyz="0 0 0" rpy="1.57079632679 0 0"/>
+      <geometry>
+        <cylinder length="0.04" radius="0.1"/>
+      </geometry>
+    </collision>
+    <inertial>
+      <mass value="1.0"/>
+      <inertia ixx="1.0" ixy="0.0" ixz="0.0" iyy="1.0" iyz="0.0" izz="1.0"/>
+    </inertial>
+  </link>
+  <joint name="base_link_wh_left_front" type="continuous">
+    <origin xyz="0.25 0.25 0" rpy="0 0 0"/>
+    <axis rpy="0 0 0" xyz="0 1 0"/>
+    <parent link="base_link"/>
+    <child link="wh_left_front"/>
+  </joint>
+  <transmission name="base_link_wh_left_front_wheel_trans">
+    <type>transmission_interface/SimpleTransmission</type>
+    <actuator name="base_link_wh_left_front_wheel_motor">
+      <mechanicalReduction>1</mechanicalReduction>
+    </actuator>
+    <joint name="base_link_wh_left_front">
+      <hardwareInterface>hardware_interface/VelocityJointInterface</hardwareInterface>
+    </joint>
+  </transmission>
+  <link name="wh_right_front">
+    <visual>
+      <origin xyz="0 0 0" rpy="1.57079632679 0 0"/>
+      <geometry>
+        <cylinder length="0.04" radius="0.1"/>
+      </geometry>
+    </visual>
+    <collision>
+      <origin xyz="0 0 0" rpy="1.57079632679 0 0"/>
+      <geometry>
+        <cylinder length="0.04" radius="0.1"/>
+      </geometry>
+    </collision>
+    <inertial>
+      <mass value="1.0"/>
+      <inertia ixx="1.0" ixy="0.0" ixz="0.0" iyy="1.0" iyz="0.0" izz="1.0"/>
+    </inertial>
+  </link>
+  <joint name="base_link_wh_right_front" type="continuous">
+    <origin xyz="0.25 -.25 0" rpy="0 0 0"/>
+    <axis rpy="0 0 0" xyz="0 1 0"/>
+    <parent link="base_link"/>
+    <child link="wh_right_front"/>
+  </joint>
+  <transmission name="base_link_wh_right_front_wheel_trans">
+    <type>transmission_interface/SimpleTransmission</type>
+    <actuator name="base_link_wh_right_front_wheel_motor">
+      <mechanicalReduction>1</mechanicalReduction>
+    </actuator>
+    <joint name="base_link_wh_right_front">
+      <hardwareInterface>hardware_interface/VelocityJointInterface</hardwareInterface>
+    </joint>
+  </transmission>
   <!-- =================== Gazebo ==================== -->
   <gazebo>
